Commit message: migrate: switch simulation stack to Gazebo Classic on Humble

File: src/external/leo_common-ros2/leo_description/urdf/macros.xacro (robot description, xacro)
@@ -452,22 +452,28 @@
           <update_rate>30</update_rate>
           <visualize>true</visualize>
-          <topic>${link_prefix}camera/image_raw</topic>
-          <ignition_frame_id>${link_prefix}camera_optical_frame</ignition_frame_id>
-          <gz_frame_id>${link_prefix}camera_optical_frame</gz_frame_id>
+          <plugin name="camera_plugin" filename="libgazebo_ros_camera.so">
+            <ros>
+              <namespace>${robot_ns}</namespace>
+              <remapping>image_raw:=camera/image_raw</remapping>
+              <remapping>camera_info:=camera/camera_info</remapping>
+            </ros>
+            <camera_name>camera</camera_name>
+            <frame_name>${link_prefix}camera_optical_frame</frame_name>
+          </plugin>
       </sensor>
     </gazebo>
-    <!-- rocker differential -->
     <gazebo>
-      <plugin name="leo_gz::DifferentialSystem" filename="libleo_gz_differential_plugin.so">
-        <jointA>rocker_L_joint</jointA>
-        <jointB>rocker_R_joint</jointB>
-        <forceConstant>100.0</forceConstant>
-      </plugin>
-    </gazebo>
-    <gazebo>
-      <plugin
-        filename="ignition-gazebo-joint-state-publisher-system"
-        name="ignition::gazebo::systems::JointStatePublisher">
-        <topic>${link_prefix}joint_states</topic>
+      <plugin name="joint_state_publisher" filename="libgazebo_ros_joint_state_publisher.so">
+        <ros>
+          <namespace>${robot_ns}</namespace>
+          <remapping>joint_states:=joint_states</remapping>
+        </ros>
+        <update_rate>50</update_rate>
+        <joint_name>wheel_FL_joint</joint_name>
+        <joint_name>wheel_FR_joint</joint_name>
+        <joint_name>wheel_RL_joint</joint_name>
+        <joint_name>wheel_RR_joint</joint_name>
+        <joint_name>rocker_L_joint</joint_name>
+        <joint_name>rocker_R_joint</joint_name>
       </plugin>
     </gazebo>
@@ -476,30 +482,38 @@
         <update_rate>100</update_rate>
         <visualize>true</visualize>
-        <topic>${link_prefix}imu/data_raw</topic>
         <always_on>1</always_on>
-        <ignition_frame_id>${link_prefix}imu_frame</ignition_frame_id>
-        <gz_frame_id>${link_prefix}imu_frame</gz_frame_id>
+        <plugin name="imu_plugin" filename="libgazebo_ros_imu_sensor.so">
+          <ros>
+            <namespace>${robot_ns}</namespace>
+            <remapping>~/out:=imu/data_raw</remapping>
+          </ros>
+        </plugin>
       </sensor>
     </gazebo>
     <gazebo>
-      <plugin
-        filename="libignition-gazebo-diff-drive-system.so"
-        name="ignition::gazebo::systems::DiffDrive">
+      <plugin name="diff_drive" filename="libgazebo_ros_diff_drive.so">
+        <ros>
+          <namespace>${robot_ns}</namespace>
+          <remapping>cmd_vel:=cmd_vel</remapping>
+          <remapping>odom:=odom</remapping>
+        </ros>
+        <num_wheel_pairs>2</num_wheel_pairs>
+        <update_rate>30</update_rate>
         <left_joint>wheel_FL_joint</left_joint>
+        <left_joint>wheel_RL_joint</left_joint>
         <right_joint>wheel_FR_joint</right_joint>
-        <left_joint>wheel_RL_joint</left_joint>
         <right_joint>wheel_RR_joint</right_joint>
         <wheel_separation>0.358</wheel_separation>
-        <wheel_radius>0.0625</wheel_radius>
-        <frame_id>odom</frame_id>
-        <child_frame_id>${link_prefix}base_footprint</child_frame_id>
-        <odom_publish_frequency>20</odom_publish_frequency>
-        <topic>${link_prefix}cmd_vel</topic>
-        <odom_topic>${link_prefix}odom</odom_topic>
-        <tf_topic>${link_prefix}tf</tf_topic>
-        <max_linear_acceleration>2.5</max_linear_acceleration>
-        <max_angular_acceleration>3</max_angular_acceleration>
-        <min_linear_acceleration>-2.5</min_linear_acceleration>
-        <min_angular_acceleration>-3</min_angular_acceleration>
+        <wheel_separation>0.358</wheel_separation>
+        <wheel_diameter>0.125</wheel_diameter>
+        <wheel_diameter>0.125</wheel_diameter>
+        <max_wheel_torque>2.0</max_wheel_torque>
+        <max_wheel_acceleration>3.0</max_wheel_acceleration>
+        <publish_odom>true</publish_odom>
+        <publish_odom_tf>true</publish_odom_tf>
+        <publish_wheel_tf>false</publish_wheel_tf>
+        <odometry_topic>odom</odometry_topic>
+        <odometry_frame>odom</odometry_frame>
+        <robot_base_frame>${link_prefix}base_footprint</robot_base_frame>
       </plugin>
     </gazebo>

File: src/lunabot_description/urdf/lunabot.urdf.xacro (robot description, xacro)
@@ -2,5 +2,5 @@
 <robot xmlns:xacro="http://ros.org/wiki/xacro" name="lunabot">
 <xacro:include filename="$(find leo_description)/urdf/leo_sim.urdf.xacro" />
-  <!-- <link name="lidar_link">
+  <link name="lidar_link">
     <visual>
       <geometry>
@@ -26,11 +26,9 @@
     <origin xyz="0.1 0.0 0.03" rpy="0 0 0"/>
   </joint>
-    <gazebo reference="lidar_link">
-    <sensor name="lidar" type="gpu_lidar">
+  <gazebo reference="lidar_link">
+    <sensor name="lidar" type="ray">
         <always_on>1</always_on>
-        <update_rate>5</update_rate>
-        <topic>scan</topic>
-        <gz_frame_id>lidar_link</gz_frame_id>
-        <lidar>
+        <update_rate>10</update_rate>
+        <ray>
         <scan>
             <horizontal>
@@ -46,21 +44,16 @@
             <resolution>0.01</resolution>
         </range>
-        </lidar>
+        </ray>
         <visualize>false</visualize>
+        <plugin name="lidar_plugin" filename="libgazebo_ros_ray_sensor.so">
+          <ros>
+            <namespace>/</namespace>
+            <remapping>~/out:=scan</remapping>
+          </ros>
+          <output_type>sensor_msgs/LaserScan</output_type>
+          <frame_name>lidar_link</frame_name>
+        </plugin>
     </sensor>
-    </gazebo> -->
-    <gazebo>
-      <plugin
-            filename="ignition-gazebo-pose-publisher-system"
-            name="ignition::gazebo::systems::PosePublisher"
-        >
-        <publish_link_poses>true</publish_link_poses>
-        <publish_sensor_poses>true</publish_sensor_poses>
-        <publish_nested_model_poses>true</publish_nested_model_poses>
-        <use_pose_vector_msg>true</use_pose_vector_msg>
-        <static_publisher>true</static_publisher>
-        <static_update_frequency>1</static_update_frequency>
-      </plugin>
-    </gazebo>
+  </gazebo>
     <link name="camera_front_link">
     <visual>
@@ -94,5 +87,5 @@
     </joint>
     <gazebo reference="camera_front_link">
-      <sensor name="camera_front" type="rgbd_camera">
+      <sensor name="camera_front" type="depth">
       <camera>
         <horizontal_fov>1.57</horizontal_fov>
@@ -108,6 +101,14 @@
       <always_on>1</always_on>
       <update_rate>10</update_rate>
-      <topic>camera_front</topic>
-        <gz_frame_id>camera_front_link</gz_frame_id>
+      <plugin name="camera_front_plugin" filename="libgazebo_ros_camera.so">
+        <ros>
+          <namespace>/</namespace>
+          <remapping>camera_front/image_raw:=camera_front/image</remapping>
+          <remapping>camera_front/depth/image_raw:=camera_front/depth_image</remapping>
+          <remapping>camera_front/points:=camera_front/points</remapping>
+        </ros>
+        <camera_name>camera_front</camera_name>
+        <frame_name>camera_front_optical_frame</frame_name>
+      </plugin>
       </sensor>
     </gazebo>
