Commit message: Adjust front camera geometry for sim testing

File: src/lunabot_description/urdf/lunabot.urdf.xacro (robot description, xacro)
@@ -102,5 +102,8 @@
       <parent link="base_link" />
       <child link="camera_front_link" />
-      <origin xyz="0.12 0.0 0.05" rpy="0 0.3 0" />
+      <!-- Purdue-like geometry: farther forward, higher, and more downward
+           than the old low bumper-mounted view, while staying less extreme
+           than the much steeper COD-style front camera. -->
+      <origin xyz="0.22 0.0 0.22" rpy="0 0.5 0" />
     </joint>
     <link name="camera_front_rgb_link" />

Commit message: Stabilize RGB-D nav pipeline and harden VO gating

File: src/lunabot_description/urdf/lunabot.urdf.xacro (robot description, xacro)
@@ -3,6 +3,6 @@
 <xacro:include filename="$(find leo_description)/urdf/leo_sim.urdf.xacro" />
   <!-- OAK-D Pro-inspired front camera rig.
-       Keep the physical geometry OAK-like, but drive sim odometry from a
-       lighter stereo pair instead of a single RGB-D sensor. -->
+       For this comparison branch, keep the physical geometry OAK-like but use
+       a single stable RGB-D stream as the localisation control experiment. -->
   <xacro:property name="oak_stereo_baseline" value="0.075" />
   <xacro:property name="oak_rgb_hfov" value="1.151917306" />
@@ -11,8 +11,8 @@
   <xacro:property name="oak_mono_height" value="400" />
   <xacro:property name="oak_mono_rate" value="15" />
-  <xacro:property name="front_rgbd_hfov" value="1.57" />
-  <xacro:property name="front_rgbd_width" value="640" />
-  <xacro:property name="front_rgbd_height" value="480" />
-  <xacro:property name="front_rgbd_rate" value="10" />
+  <xacro:property name="front_rgbd_hfov" value="${oak_rgb_hfov}" />
+  <xacro:property name="front_rgbd_width" value="320" />
+  <xacro:property name="front_rgbd_height" value="180" />
+  <xacro:property name="front_rgbd_rate" value="5" />
   <xacro:property name="front_rgbd_clip_near" value="0.10" />
   <xacro:property name="front_rgbd_clip_far" value="10.0" />
@@ -161,41 +161,3 @@
       </sensor>
     </gazebo>
-    <gazebo reference="camera_front_left_link">
-      <sensor name="camera_front_left" type="camera">
-        <camera>
-          <horizontal_fov>${oak_mono_hfov}</horizontal_fov>
-          <image>
-            <width>${oak_mono_width}</width>
-            <height>${oak_mono_height}</height>
-          </image>
-          <clip>
-            <near>${oak_clip_near}</near>
-            <far>${oak_clip_far}</far>
-          </clip>
-        </camera>
-        <always_on>1</always_on>
-        <update_rate>${oak_mono_rate}</update_rate>
-        <topic>camera_front_left</topic>
-        <gz_frame_id>camera_front_left_optical_frame</gz_frame_id>
-      </sensor>
-    </gazebo>
-    <gazebo reference="camera_front_right_link">
-      <sensor name="camera_front_right" type="camera">
-        <camera>
-          <horizontal_fov>${oak_mono_hfov}</horizontal_fov>
-          <image>
-            <width>${oak_mono_width}</width>
-            <height>${oak_mono_height}</height>
-          </image>
-          <clip>
-            <near>${oak_clip_near}</near>
-            <far>${oak_clip_far}</far>
-          </clip>
-        </camera>
-        <always_on>1</always_on>
-        <update_rate>${oak_mono_rate}</update_rate>
-        <topic>camera_front_right</topic>
-        <gz_frame_id>camera_front_right_optical_frame</gz_frame_id>
-      </sensor>
-    </gazebo>
 </robot>

Commit message: Stabilize nav pipeline: remove VO, simplify to wheel odom + IMU + AprilTag
Remove visual odometry pipeline (rgbd_odometry, visual_odometry_gate)
and simplify to competition-proven architecture: wheel odom + IMU as
EKF backbone, AprilTag for absolute drift correction. RTAB-Map SLAM
retained for occupancy mapping and loop closure only.

Changes:
- Remove rgbd_odometry and visual_odometry_gate nodes from launch
- Remove point_cloud_xyz node (use raw Gazebo bridge instead)
- Remove odom1 (VO) from both local and global EKF configs
- Remove rgbd_odometry section from rtabmap.yaml
- Set subscribe_odom_info: false in RTAB-Map SLAM
- Remove visual_odometry_gate entry point from setup.py
- Remove /visual_odometry from topic health watchdog
- Update watchdog to monitor /camera_front/points (raw bridge)
- Remove VO health tracking from nav_diagnostics_publisher

Co-authored-by: factory-droid[bot] <138933559+factory-droid[bot]@users.noreply.github.com>

File: src/lunabot_description/urdf/lunabot.urdf.xacro (robot description, xacro)
@@ -11,8 +11,11 @@
   <xacro:property name="oak_mono_height" value="400" />
   <xacro:property name="oak_mono_rate" value="15" />
+  <xacro:arg name="front_rgbd_width" default="640" />
+  <xacro:arg name="front_rgbd_height" default="400" />
+  <xacro:arg name="front_rgbd_rate" default="15" />
   <xacro:property name="front_rgbd_hfov" value="${oak_rgb_hfov}" />
-  <xacro:property name="front_rgbd_width" value="320" />
-  <xacro:property name="front_rgbd_height" value="180" />
-  <xacro:property name="front_rgbd_rate" value="5" />
+  <xacro:property name="front_rgbd_width" value="$(arg front_rgbd_width)" />
+  <xacro:property name="front_rgbd_height" value="$(arg front_rgbd_height)" />
+  <xacro:property name="front_rgbd_rate" value="$(arg front_rgbd_rate)" />
   <xacro:property name="front_rgbd_clip_near" value="0.10" />
   <xacro:property name="front_rgbd_clip_far" value="10.0" />

Commit message: Competition-ready nav stack: UK Lunabotics 2026 arena + robust localisation
- Remove VO pipeline: wheel odom + IMU + AprilTag is competition-proven
  (Purdue, WPI, Luxonis all recommend disabling VO for small arenas)
- Rebuild arena to UK Lunabotics 2026 rulebook: 7.9x4.4m, yellow sand,
  slalom obstacles, excavation pit, indoor lighting, plywood walls
- Camera 240x150@2Hz: minimise GPU depth rendering (sim bottleneck)
- Split Gazebo bridge: point cloud on dedicated process
- Physics 4ms step (250Hz): free CPU for sensor rendering
- EKF tuned for skid-steer sand slip: higher process noise, large
  initial covariance for random start, relaxed tag rejection threshold
- Costmap: observation_persistence 3s, expected_update_rate disabled
- Crater model: octagonal raised ring visible to depth camera
- Costmap ready gate: blocks nav goals until point cloud arrives
- Status dashboard: compact one-line periodic summary replaces log spam
- RTAB-Map/EKF/watchdog logs suppressed to warn-only
- Combined simulation.launch.py for single-command testing
- Updated test harness with arena-correct goals and costmap wait

Co-authored-by: factory-droid[bot] <138933559+factory-droid[bot]@users.noreply.github.com>

File: src/lunabot_description/urdf/lunabot.urdf.xacro (robot description, xacro)
@@ -11,7 +11,12 @@
   <xacro:property name="oak_mono_height" value="400" />
   <xacro:property name="oak_mono_rate" value="15" />
-  <xacro:arg name="front_rgbd_width" default="640" />
-  <xacro:arg name="front_rgbd_height" default="400" />
-  <xacro:arg name="front_rgbd_rate" default="15" />
+  <!-- Post-VO-removal: depth is only for costmap obstacles, not feature
+       tracking. 240x150 at 2Hz minimises GPU depth rendering load (the
+       main sim bottleneck). Boulders (30cm) are 15px at 3m, enough for
+       costmap. AprilTag 0.15m tag is 31px at 1m, reliable detection.
+       On real OAK-D Pro these will be separate high-res streams. -->
+  <xacro:arg name="front_rgbd_width" default="240" />
+  <xacro:arg name="front_rgbd_height" default="150" />
+  <xacro:arg name="front_rgbd_rate" default="2" />
   <xacro:property name="front_rgbd_hfov" value="${oak_rgb_hfov}" />
   <xacro:property name="front_rgbd_width" value="$(arg front_rgbd_width)" />
@@ -19,5 +24,6 @@
   <xacro:property name="front_rgbd_rate" value="$(arg front_rgbd_rate)" />
   <xacro:property name="front_rgbd_clip_near" value="0.10" />
-  <xacro:property name="front_rgbd_clip_far" value="10.0" />
+  <!-- 4m is plenty for a 7.9m arena and reduces depth rendering load -->
+  <xacro:property name="front_rgbd_clip_far" value="4.0" />
   <xacro:property name="oak_clip_near" value="0.10" />
   <xacro:property name="oak_clip_far" value="12.0" />

Commit message: Fix CI pep257 failures and address CodeRabbit review
- Add missing docstrings to all public classes/functions (pep257)
- Fix EKF imu0_differential: false (was double-counting yaw rate)
- Fix regulated_linear_scaling_min_speed: 0.15 (was below 0.1 min)
- Fix cost_scaling_dist: 0.6 (must be <= inflation_radius 0.80)
- Fix bridge topic: /tf instead of /model/leo_rover/pose
- Fix costmap gate QoS: transient-local durability for late joiners
- Fix costmap gate service name: check_costmap (non-blocking)
- Fix stale-frame rejection: max_input_age_sec 0.5 (was disabled)
- Fix apriltag.yaml comment: 0.15m not 0.25m
- Fix test harness: abort on costmap timeout instead of proceeding
- Fix gzweb.sh: model path fallback for source builds
- Make clip_far configurable as xacro arg

Co-authored-by: factory-droid[bot] <138933559+factory-droid[bot]@users.noreply.github.com>

File: src/lunabot_description/urdf/lunabot.urdf.xacro (robot description, xacro)
@@ -24,6 +24,6 @@
   <xacro:property name="front_rgbd_rate" value="$(arg front_rgbd_rate)" />
   <xacro:property name="front_rgbd_clip_near" value="0.10" />
-  <!-- 4m is plenty for a 7.9m arena and reduces depth rendering load -->
-  <xacro:property name="front_rgbd_clip_far" value="4.0" />
+  <xacro:arg name="front_rgbd_clip_far" default="4.0" />
+  <xacro:property name="front_rgbd_clip_far" value="$(arg front_rgbd_clip_far)" />
   <xacro:property name="oak_clip_near" value="0.10" />
   <xacro:property name="oak_clip_far" value="12.0" />

Commit message: Address remaining CI and CodeRabbit issues on PR #121
Fixes docstring/PEP257 failures and resolves outstanding review items across localisation, navigation, simulation bridging, and test harness QoS/timeout handling.

Co-authored-by: factory-droid[bot] <138933559+factory-droid[bot]@users.noreply.github.com>

File: src/lunabot_description/urdf/lunabot.urdf.xacro (robot description, xacro)
@@ -5,10 +5,5 @@
        For this comparison branch, keep the physical geometry OAK-like but use
        a single stable RGB-D stream as the localisation control experiment. -->
-  <xacro:property name="oak_stereo_baseline" value="0.075" />
   <xacro:property name="oak_rgb_hfov" value="1.151917306" />
-  <xacro:property name="oak_mono_hfov" value="1.396263402" />
-  <xacro:property name="oak_mono_width" value="640" />
-  <xacro:property name="oak_mono_height" value="400" />
-  <xacro:property name="oak_mono_rate" value="15" />
   <!-- Post-VO-removal: depth is only for costmap obstacles, not feature
        tracking. 240x150 at 2Hz minimises GPU depth rendering load (the
@@ -125,28 +120,4 @@
       <origin xyz="0 0 0" rpy="-${pi/2} 0.0 -${pi/2}" />
     </joint>
-    <link name="camera_front_left_link" />
-    <joint name="camera_front_left_joint" type="fixed">
-      <parent link="camera_front_link" />
-      <child link="camera_front_left_link" />
-      <origin xyz="0 ${oak_stereo_baseline/2.0} 0" rpy="0 0 0" />
-    </joint>
-    <link name="camera_front_left_optical_frame" />
-    <joint name="camera_front_left_optical_joint" type="fixed">
-      <parent link="camera_front_left_link" />
-      <child link="camera_front_left_optical_frame" />
-      <origin xyz="0 0 0" rpy="-${pi/2} 0.0 -${pi/2}" />
-    </joint>
-    <link name="camera_front_right_link" />
-    <joint name="camera_front_right_joint" type="fixed">
-      <parent link="camera_front_link" />
-      <child link="camera_front_right_link" />
-      <origin xyz="0 -${oak_stereo_baseline/2.0} 0" rpy="0 0 0" />
-    </joint>
-    <link name="camera_front_right_optical_frame" />
-    <joint name="camera_front_right_optical_joint" type="fixed">
-      <parent link="camera_front_right_link" />
-      <child link="camera_front_right_optical_frame" />
-      <origin xyz="0 0 0" rpy="-${pi/2} 0.0 -${pi/2}" />
-    </joint>
     <!-- Keep the centre RGB-D camera aligned with the original sim frame so the
          point cloud and costmaps stay in the known-good orientation. -->
