Commit message: Reset sim baseline around lightweight rover and world

File: src/lunabot_description/urdf/lunabot.urdf.xacro (robot description, xacro)
@@ -1,15 +1,14 @@
-<?xml version="1.0" ?>
+<?xml version="1.0"?>
 <robot xmlns:xacro="http://ros.org/wiki/xacro" name="lunabot">
-<xacro:include filename="$(find leo_description)/urdf/leo_sim.urdf.xacro" />
-  <!-- OAK-D Pro-inspired front camera rig.
-       Keep the physical geometry OAK-like, but drive sim odometry from a
-       lighter stereo pair instead of a single RGB-D sensor. -->
-  <xacro:property name="oak_stereo_baseline" value="0.075" />
-  <xacro:property name="oak_rgb_hfov" value="1.151917306" />
-  <xacro:property name="oak_mono_hfov" value="1.396263402" />
-  <xacro:property name="oak_mono_width" value="640" />
-  <xacro:property name="oak_mono_height" value="400" />
-  <xacro:property name="oak_mono_rate" value="15" />
-  <xacro:property name="front_rgbd_hfov" value="1.57" />
+  <xacro:property name="chassis_length" value="0.82" />
+  <xacro:property name="chassis_width" value="0.58" />
+  <xacro:property name="chassis_height" value="0.16" />
+  <xacro:property name="wheel_radius" value="0.14" />
+  <xacro:property name="wheel_width" value="0.08" />
+  <xacro:property name="wheel_x" value="0.26" />
+  <xacro:property name="wheel_y" value="0.26" />
+  <xacro:property name="wheel_z" value="-0.12" />
+  <xacro:property name="wheel_separation" value="0.52" />
+  <xacro:property name="front_rgbd_hfov" value="1.15" />
   <xacro:property name="front_rgbd_width" value="640" />
   <xacro:property name="front_rgbd_height" value="480" />
@@ -17,79 +16,162 @@
   <xacro:property name="front_rgbd_clip_near" value="0.10" />
   <xacro:property name="front_rgbd_clip_far" value="10.0" />
-  <xacro:property name="oak_clip_near" value="0.10" />
-  <xacro:property name="oak_clip_far" value="12.0" />
-  <!-- <link name="lidar_link">
-    <visual>
-      <geometry>
-        <cylinder length="0.05" radius="0.03"/>
-      </geometry>
-      <material name="dark_grey">
-        <color rgba="0.2 0.2 0.2 1.0"/>
-      </material>
-    </visual>
-    <collision>
-      <geometry>
-        <cylinder length="0.05" radius="0.03"/>
-      </geometry>
-    </collision>
-    <inertial>
-      <mass value="0.1"/>
-      <inertia ixx="0.0001" ixy="0" ixz="0" iyy="0.0001" iyz="0" izz="0.0001"/>
-    </inertial>
-  </link>
-  <joint name="lidar_joint" type="fixed">
-    <parent link="base_link"/>
-    <child link="lidar_link"/>
-    <origin xyz="0.1 0.0 0.03" rpy="0 0 0"/>
-  </joint>
-    <gazebo reference="lidar_link">
-    <sensor name="lidar" type="gpu_lidar">
-        <always_on>1</always_on>
-        <update_rate>5</update_rate>
-        <topic>scan</topic>
-        <gz_frame_id>lidar_link</gz_frame_id>
-        <lidar>
-        <scan>
-            <horizontal>
-            <samples>180</samples>
-            <resolution>1</resolution>
-            <min_angle>-3.14159</min_angle>
-            <max_angle>3.14159</max_angle>
-            </horizontal>
-        </scan>
-        <range>
-            <min>0.1</min>
-            <max>10.0</max>
-            <resolution>0.01</resolution>
-        </range>
-        </lidar>
-        <visualize>false</visualize>
-    </sensor>
-    </gazebo> -->
-    <gazebo>
-      <plugin
-            filename="ignition-gazebo-pose-publisher-system"
-            name="ignition::gazebo::systems::PosePublisher"
-        >
-        <publish_link_poses>true</publish_link_poses>
-        <publish_sensor_poses>true</publish_sensor_poses>
-        <publish_nested_model_poses>true</publish_nested_model_poses>
-        <use_pose_vector_msg>true</use_pose_vector_msg>
-        <static_publisher>true</static_publisher>
-        <static_update_frequency>1</static_update_frequency>
-      </plugin>
-    </gazebo>
-    <link name="camera_front_link">
-    <visual>
-      <geometry>
-        <box size="0.09 0.04 0.03" />
-      </geometry>
-      <material name="dark_grey">
-        <color rgba="0.2 0.2 0.2 1.0" />
-      </material>
-    </visual>
-    <collision>
-      <geometry>
-        <box size="0.09 0.04 0.03" />
+  <material name="sand_beige">
+    <color rgba="0.71 0.62 0.44 1.0" />
+  </material>
+  <material name="dark_grey">
+    <color rgba="0.18 0.18 0.20 1.0" />
+  </material>
+  <link name="base_footprint" />
+  <link name="base_link">
+    <inertial>
+      <origin xyz="0 0 0" rpy="0 0 0" />
+      <mass value="45.0" />
+      <inertia
+        ixx="2.2"
+        ixy="0.0"
+        ixz="0.0"
+        iyy="2.9"
+        iyz="0.0"
+        izz="4.3" />
+    </inertial>
+    <visual>
+      <origin xyz="0 0 0.03" rpy="0 0 0" />
+      <geometry>
+        <box size="${chassis_length} ${chassis_width} ${chassis_height}" />
+      </geometry>
+      <material name="sand_beige" />
+    </visual>
+    <collision>
+      <origin xyz="0 0 0.03" rpy="0 0 0" />
+      <geometry>
+        <box size="${chassis_length} ${chassis_width} ${chassis_height}" />
+      </geometry>
+    </collision>
+  </link>
+  <joint name="base_footprint_joint" type="fixed">
+    <parent link="base_footprint" />
+    <child link="base_link" />
+    <origin xyz="0 0 ${wheel_radius}" rpy="0 0 0" />
+  </joint>
+  <link name="imu_frame" />
+  <joint name="imu_joint" type="fixed">
+    <parent link="base_link" />
+    <child link="imu_frame" />
+    <origin xyz="0 0 0.04" rpy="0 0 0" />
+  </joint>
+  <link name="wheel_front_left">
+    <inertial>
+      <origin xyz="0 0 0" rpy="0 0 0" />
+      <mass value="3.0" />
+      <inertia ixx="0.03" ixy="0.0" ixz="0.0" iyy="0.03" iyz="0.0" izz="0.03" />
+    </inertial>
+    <visual>
+      <origin xyz="0 0 0" rpy="1.57079632679 0 0" />
+      <geometry>
+        <cylinder radius="${wheel_radius}" length="${wheel_width}" />
+      </geometry>
+      <material name="dark_grey" />
+    </visual>
+    <collision>
+      <origin xyz="0 0 0" rpy="1.57079632679 0 0" />
+      <geometry>
+        <cylinder radius="${wheel_radius}" length="${wheel_width}" />
+      </geometry>
+    </collision>
+  </link>
+  <link name="wheel_front_right">
+    <inertial>
+      <origin xyz="0 0 0" rpy="0 0 0" />
+      <mass value="3.0" />
+      <inertia ixx="0.03" ixy="0.0" ixz="0.0" iyy="0.03" iyz="0.0" izz="0.03" />
+    </inertial>
+    <visual>
+      <origin xyz="0 0 0" rpy="1.57079632679 0 0" />
+      <geometry>
+        <cylinder radius="${wheel_radius}" length="${wheel_width}" />
+      </geometry>
+      <material name="dark_grey" />
+    </visual>
+    <collision>
+      <origin xyz="0 0 0" rpy="1.57079632679 0 0" />
+      <geometry>
+        <cylinder radius="${wheel_radius}" length="${wheel_width}" />
+      </geometry>
+    </collision>
+  </link>
+  <link name="wheel_rear_left">
+    <inertial>
+      <origin xyz="0 0 0" rpy="0 0 0" />
+      <mass value="3.0" />
+      <inertia ixx="0.03" ixy="0.0" ixz="0.0" iyy="0.03" iyz="0.0" izz="0.03" />
+    </inertial>
+    <visual>
+      <origin xyz="0 0 0" rpy="1.57079632679 0 0" />
+      <geometry>
+        <cylinder radius="${wheel_radius}" length="${wheel_width}" />
+      </geometry>
+      <material name="dark_grey" />
+    </visual>
+    <collision>
+      <origin xyz="0 0 0" rpy="1.57079632679 0 0" />
+      <geometry>
+        <cylinder radius="${wheel_radius}" length="${wheel_width}" />
+      </geometry>
+    </collision>
+  </link>
+  <link name="wheel_rear_right">
+    <inertial>
+      <origin xyz="0 0 0" rpy="0 0 0" />
+      <mass value="3.0" />
+      <inertia ixx="0.03" ixy="0.0" ixz="0.0" iyy="0.03" iyz="0.0" izz="0.03" />
+    </inertial>
+    <visual>
+      <origin xyz="0 0 0" rpy="1.57079632679 0 0" />
+      <geometry>
+        <cylinder radius="${wheel_radius}" length="${wheel_width}" />
+      </geometry>
+      <material name="dark_grey" />
+    </visual>
+    <collision>
+      <origin xyz="0 0 0" rpy="1.57079632679 0 0" />
+      <geometry>
+        <cylinder radius="${wheel_radius}" length="${wheel_width}" />
+      </geometry>
+    </collision>
+  </link>
+  <joint name="wheel_front_left_joint" type="continuous">
+    <parent link="base_link" />
+    <child link="wheel_front_left" />
+    <origin xyz="${wheel_x} ${wheel_y} ${wheel_z}" rpy="0 0 0" />
+    <axis xyz="0 1 0" />
+  </joint>
+  <joint name="wheel_front_right_joint" type="continuous">
+    <parent link="base_link" />
+    <child link="wheel_front_right" />
+    <origin xyz="${wheel_x} -${wheel_y} ${wheel_z}" rpy="0 0 0" />
+    <axis xyz="0 1 0" />
+  </joint>
+  <joint name="wheel_rear_left_joint" type="continuous">
+    <parent link="base_link" />
+    <child link="wheel_rear_left" />
+    <origin xyz="-${wheel_x} ${wheel_y} ${wheel_z}" rpy="0 0 0" />
+    <axis xyz="0 1 0" />
+  </joint>
+  <joint name="wheel_rear_right_joint" type="continuous">
+    <parent link="base_link" />
+    <child link="wheel_rear_right" />
+    <origin xyz="-${wheel_x} -${wheel_y} ${wheel_z}" rpy="0 0 0" />
+    <axis xyz="0 1 0" />
+  </joint>
+  <link name="camera_front_link">
+    <visual>
+      <geometry>
+        <box size="0.10 0.04 0.03" />
+      </geometry>
+      <material name="dark_grey" />
+    </visual>
+    <collision>
+      <geometry>
+        <box size="0.10 0.04 0.03" />
       </geometry>
     </collision>
@@ -99,103 +181,86 @@
     </inertial>
   </link>
-    <joint name="camera_front_joint" type="fixed">
-      <parent link="base_link" />
-      <child link="camera_front_link" />
-      <origin xyz="0.12 0.0 0.05" rpy="0 0.3 0" />
-    </joint>
-    <link name="camera_front_rgb_link" />
-    <joint name="camera_front_rgb_joint" type="fixed">
-      <parent link="camera_front_link" />
-      <child link="camera_front_rgb_link" />
-      <origin xyz="0 0 0" rpy="0 0 0" />
-    </joint>
-    <link name="camera_front_optical_frame" />
-    <joint name="camera_front_optical_joint" type="fixed">
-      <parent link="camera_front_rgb_link" />
-      <child link="camera_front_optical_frame" />
-      <origin xyz="0 0 0" rpy="-${pi/2} 0.0 -${pi/2}" />
-    </joint>
-    <link name="camera_front_left_link" />
-    <joint name="camera_front_left_joint" type="fixed">
-      <parent link="camera_front_link" />
-      <child link="camera_front_left_link" />
-      <origin xyz="0 ${oak_stereo_baseline/2.0} 0" rpy="0 0 0" />
-    </joint>
-    <link name="camera_front_left_optical_frame" />
-    <joint name="camera_front_left_optical_joint" type="fixed">
-      <parent link="camera_front_left_link" />
-      <child link="camera_front_left_optical_frame" />
-      <origin xyz="0 0 0" rpy="-${pi/2} 0.0 -${pi/2}" />
-    </joint>
-    <link name="camera_front_right_link" />
-    <joint name="camera_front_right_joint" type="fixed">
-      <parent link="camera_front_link" />
-      <child link="camera_front_right_link" />
-      <origin xyz="0 -${oak_stereo_baseline/2.0} 0" rpy="0 0 0" />
-    </joint>
-    <link name="camera_front_right_optical_frame" />
-    <joint name="camera_front_right_optical_joint" type="fixed">
-      <parent link="camera_front_right_link" />
-      <child link="camera_front_right_optical_frame" />
-      <origin xyz="0 0 0" rpy="-${pi/2} 0.0 -${pi/2}" />
-    </joint>
-    <!-- Keep the centre RGB-D camera aligned with the original sim frame so the
-         point cloud and costmaps stay in the known-good orientation. -->
-    <gazebo reference="camera_front_link">
-      <sensor name="camera_front" type="rgbd_camera">
-        <camera>
-          <horizontal_fov>${front_rgbd_hfov}</horizontal_fov>
-          <image>
-            <width>${front_rgbd_width}</width>
-            <height>${front_rgbd_height}</height>
-          </image>
-          <clip>
-            <near>${front_rgbd_clip_near}</near>
-            <far>${front_rgbd_clip_far}</far>
-          </clip>
-        </camera>
-        <always_on>1</always_on>
-        <update_rate>${front_rgbd_rate}</update_rate>
-        <topic>camera_front</topic>
-        <gz_frame_id>camera_front_link</gz_frame_id>
-      </sensor>
-    </gazebo>
-    <gazebo reference="camera_front_left_link">
-      <sensor name="camera_front_left" type="camera">
-        <camera>
-          <horizontal_fov>${oak_mono_hfov}</horizontal_fov>
-          <image>
-            <width>${oak_mono_width}</width>
-            <height>${oak_mono_height}</height>
-          </image>
-          <clip>
-            <near>${oak_clip_near}</near>
-            <far>${oak_clip_far}</far>
-          </clip>
-        </camera>
-        <always_on>1</always_on>
-        <update_rate>${oak_mono_rate}</update_rate>
-        <topic>camera_front_left</topic>
-        <gz_frame_id>camera_front_left_optical_frame</gz_frame_id>
-      </sensor>
-    </gazebo>
-    <gazebo reference="camera_front_right_link">
-      <sensor name="camera_front_right" type="camera">
-        <camera>
-          <horizontal_fov>${oak_mono_hfov}</horizontal_fov>
-          <image>
-            <width>${oak_mono_width}</width>
-            <height>${oak_mono_height}</height>
-          </image>
-          <clip>
-            <near>${oak_clip_near}</near>
-            <far>${oak_clip_far}</far>
-          </clip>
-        </camera>
-        <always_on>1</always_on>
-        <update_rate>${oak_mono_rate}</update_rate>
-        <topic>camera_front_right</topic>
-        <gz_frame_id>camera_front_right_optical_frame</gz_frame_id>
-      </sensor>
-    </gazebo>
+  <joint name="camera_front_joint" type="fixed">
+    <parent link="base_link" />
+    <child link="camera_front_link" />
+    <origin xyz="0.26 0.0 0.14" rpy="0 0.18 0" />
+  </joint>
+  <link name="camera_front_optical_frame" />
+  <joint name="camera_front_optical_joint" type="fixed">
+    <parent link="camera_front_link" />
+    <child link="camera_front_optical_frame" />
+    <origin xyz="0 0 0" rpy="-${pi/2} 0.0 -${pi/2}" />
+  </joint>
+  <gazebo>
+    <plugin
+      filename="ignition-gazebo-joint-state-publisher-system"
+      name="ignition::gazebo::systems::JointStatePublisher">
+      <topic>joint_states</topic>
+    </plugin>
+  </gazebo>
+  <gazebo reference="imu_frame">
+    <sensor type="imu" name="lunabot_imu_sensor">
+      <always_on>1</always_on>
+      <update_rate>100</update_rate>
+      <topic>imu/data_raw</topic>
+      <gz_frame_id>imu_frame</gz_frame_id>
+    </sensor>
+  </gazebo>
+  <gazebo reference="camera_front_link">
+    <sensor name="camera_front" type="rgbd_camera">
+      <always_on>1</always_on>
+      <update_rate>${front_rgbd_rate}</update_rate>
+      <topic>camera_front</topic>
+      <gz_frame_id>camera_front_optical_frame</gz_frame_id>
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
Commit message: Trim sim camera load for baseline rover

File: src/lunabot_description/urdf/lunabot.urdf.xacro (robot description, xacro)
@@ -11,6 +11,6 @@
   <xacro:property name="wheel_separation" value="0.52" />
   <xacro:property name="front_rgbd_hfov" value="1.15" />
-  <xacro:property name="front_rgbd_width" value="640" />
-  <xacro:property name="front_rgbd_height" value="480" />
+  <xacro:property name="front_rgbd_width" value="424" />
+  <xacro:property name="front_rgbd_height" value="240" />
   <xacro:property name="front_rgbd_rate" value="10" />
   <xacro:property name="front_rgbd_clip_near" value="0.10" />

Commit message: Align sim RGB-D sensor with optical frame

File: src/lunabot_description/urdf/lunabot.urdf.xacro (robot description, xacro)
@@ -186,9 +186,15 @@
     <origin xyz="0.26 0.0 0.14" rpy="0 0.18 0" />
   </joint>
+  <link name="camera_front_rgb_link" />
+  <joint name="camera_front_rgb_joint" type="fixed">
+    <parent link="camera_front_link" />
+    <child link="camera_front_rgb_link" />
+    <origin xyz="0 0 0" rpy="-${pi/2} 0.0 -${pi/2}" />
+  </joint>
   <link name="camera_front_optical_frame" />
   <joint name="camera_front_optical_joint" type="fixed">
-    <parent link="camera_front_link" />
+    <parent link="camera_front_rgb_link" />
     <child link="camera_front_optical_frame" />
-    <origin xyz="0 0 0" rpy="-${pi/2} 0.0 -${pi/2}" />
+    <origin xyz="0 0 0" rpy="0 0 0" />
   </joint>
   <gazebo>
@@ -207,5 +213,5 @@
     </sensor>
   </gazebo>
-  <gazebo reference="camera_front_link">
+  <gazebo reference="camera_front_rgb_link">
     <sensor name="camera_front" type="rgbd_camera">
       <always_on>1</always_on>

Commit message: Restore forward-facing sim camera mount

File: src/lunabot_description/urdf/lunabot.urdf.xacro (robot description, xacro)
@@ -184,5 +184,5 @@
     <parent link="base_link" />
     <child link="camera_front_link" />
-    <origin xyz="0.26 0.0 0.14" rpy="0 0.18 0" />
+    <origin xyz="0.48 0.0 0.20" rpy="0 0.10 0" />
   </joint>
   <link name="camera_front_rgb_link" />
@@ -190,5 +190,5 @@
     <parent link="camera_front_link" />
     <child link="camera_front_rgb_link" />
-    <origin xyz="0 0 0" rpy="-${pi/2} 0.0 -${pi/2}" />
+    <origin xyz="0 0 0" rpy="0 0 0" />
   </joint>
   <link name="camera_front_optical_frame" />
@@ -196,5 +196,5 @@
     <parent link="camera_front_rgb_link" />
     <child link="camera_front_optical_frame" />
-    <origin xyz="0 0 0" rpy="0 0 0" />
+    <origin xyz="0 0 0" rpy="-${pi/2} 0.0 -${pi/2}" />
   </joint>
   <gazebo>
@@ -213,10 +213,10 @@
     </sensor>
   </gazebo>
-  <gazebo reference="camera_front_rgb_link">
+  <gazebo reference="camera_front_link">
     <sensor name="camera_front" type="rgbd_camera">
       <always_on>1</always_on>
       <update_rate>${front_rgbd_rate}</update_rate>
       <topic>camera_front</topic>
-      <gz_frame_id>camera_front_optical_frame</gz_frame_id>
+      <gz_frame_id>camera_front_link</gz_frame_id>
       <camera>
         <horizontal_fov>${front_rgbd_hfov}</horizontal_fov>

Commit message: sim: add ouster mount and bridge plumbing

File: src/lunabot_description/urdf/lunabot.urdf.xacro (robot description, xacro)
@@ -2,8 +2,8 @@
 <robot xmlns:xacro="http://ros.org/wiki/xacro" name="lunabot">
 <xacro:include filename="$(find leo_description)/urdf/leo_sim.urdf.xacro" />
-  <!-- <link name="lidar_link">
+  <link name="ouster_link">
     <visual>
       <geometry>
-        <cylinder length="0.05" radius="0.03"/>
+        <cylinder length="0.08" radius="0.05"/>
       </geometry>
       <material name="dark_grey">
@@ -17,37 +17,43 @@
     </collision>
     <inertial>
-      <mass value="0.1"/>
-      <inertia ixx="0.0001" ixy="0" ixz="0" iyy="0.0001" iyz="0" izz="0.0001"/>
+      <mass value="0.8"/>
+      <inertia ixx="0.001" ixy="0" ixz="0" iyy="0.001" iyz="0" izz="0.001"/>
     </inertial>
   </link>
-  <joint name="lidar_joint" type="fixed">
+  <joint name="ouster_joint" type="fixed">
     <parent link="base_link"/>
-    <child link="lidar_link"/>
-    <origin xyz="0.1 0.0 0.03" rpy="0 0 0"/>
+    <child link="ouster_link"/>
+    <origin xyz="0.0 0.0 0.24" rpy="0 0 0"/>
   </joint>
-    <gazebo reference="lidar_link">
-    <sensor name="lidar" type="gpu_lidar">
+    <gazebo reference="ouster_link">
+    <sensor name="ouster" type="gpu_lidar">
         <always_on>1</always_on>
-        <update_rate>5</update_rate>
-        <topic>scan</topic>
-        <gz_frame_id>lidar_link</gz_frame_id>
+        <update_rate>10</update_rate>
+        <topic>ouster/points</topic>
+        <gz_frame_id>ouster_link</gz_frame_id>
         <lidar>
         <scan>
             <horizontal>
-            <samples>180</samples>
+            <samples>1024</samples>
             <resolution>1</resolution>
             <min_angle>-3.14159</min_angle>
             <max_angle>3.14159</max_angle>
             </horizontal>
+            <vertical>
+            <samples>16</samples>
+            <resolution>1</resolution>
+            <min_angle>-0.261799</min_angle>
+            <max_angle>0.261799</max_angle>
+            </vertical>
         </scan>
         <range>
-            <min>0.1</min>
-            <max>10.0</max>
-            <resolution>0.01</resolution>
+            <min>0.3</min>
+            <max>20.0</max>
+            <resolution>0.02</resolution>
         </range>
         </lidar>
         <visualize>false</visualize>
     </sensor>
-    </gazebo> -->
+    </gazebo>
     <gazebo>
       <plugin

Commit message: sim: make ouster mount non-invasive and visible

File: src/lunabot_description/urdf/lunabot.urdf.xacro (robot description, xacro)
@@ -4,19 +4,15 @@
   <link name="ouster_link">
     <visual>
+      <origin xyz="0 0 0.015" rpy="0 0 0"/>
       <geometry>
-        <cylinder length="0.08" radius="0.05"/>
+        <box size="0.09 0.09 0.03"/>
       </geometry>
-      <material name="dark_grey">
-        <color rgba="0.2 0.2 0.2 1.0"/>
+      <material name="sensor_black">
+        <color rgba="0.05 0.05 0.05 1.0"/>
       </material>
     </visual>
-    <collision>
-      <geometry>
-        <cylinder length="0.05" radius="0.03"/>
-      </geometry>
-    </collision>
     <inertial>
-      <mass value="0.8"/>
-      <inertia ixx="0.001" ixy="0" ixz="0" iyy="0.001" iyz="0" izz="0.001"/>
+      <mass value="0.001"/>
+      <inertia ixx="1e-6" ixy="0" ixz="0" iyy="1e-6" iyz="0" izz="1e-6"/>
     </inertial>
   </link>
@@ -24,5 +20,5 @@
     <parent link="base_link"/>
     <child link="ouster_link"/>
-    <origin xyz="0.0 0.0 0.24" rpy="0 0 0"/>
+    <origin xyz="0.0 0.0 0.30" rpy="0 0 0"/>
   </joint>
     <gazebo reference="ouster_link">

Commit message: sim: use cylindrical visual for ouster mount

File: src/lunabot_description/urdf/lunabot.urdf.xacro (robot description, xacro)
@@ -4,7 +4,7 @@
   <link name="ouster_link">
     <visual>
-      <origin xyz="0 0 0.015" rpy="0 0 0"/>
+      <origin xyz="0 0 0.03" rpy="0 0 0"/>
       <geometry>
-        <box size="0.09 0.09 0.03"/>
+        <cylinder length="0.06" radius="0.035"/>
       </geometry>
       <material name="sensor_black">
