Commit message: sim: add ouster mount and bridge plumbing (#132)
* sim: add ouster mount and bridge plumbing

* sim: make ouster mount non-invasive and visible

* sim: bridge ouster point cloud transport topic

* sim: use cylindrical visual for ouster mount

File: src/lunabot_description/urdf/lunabot.urdf.xacro (robot description, xacro)
@@ -2,52 +2,54 @@
 <robot xmlns:xacro="http://ros.org/wiki/xacro" name="lunabot">
 <xacro:include filename="$(find leo_description)/urdf/leo_sim.urdf.xacro" />
-  <!-- <link name="lidar_link">
+  <link name="ouster_link">
     <visual>
+      <origin xyz="0 0 0.03" rpy="0 0 0"/>
       <geometry>
-        <cylinder length="0.05" radius="0.03"/>
+        <cylinder length="0.06" radius="0.035"/>
       </geometry>
-      <material name="dark_grey">
-        <color rgba="0.2 0.2 0.2 1.0"/>
+      <material name="sensor_black">
+        <color rgba="0.05 0.05 0.05 1.0"/>
       </material>
     </visual>
-    <collision>
-      <geometry>
-        <cylinder length="0.05" radius="0.03"/>
-      </geometry>
-    </collision>
     <inertial>
-      <mass value="0.1"/>
-      <inertia ixx="0.0001" ixy="0" ixz="0" iyy="0.0001" iyz="0" izz="0.0001"/>
+      <mass value="0.001"/>
+      <inertia ixx="1e-6" ixy="0" ixz="0" iyy="1e-6" iyz="0" izz="1e-6"/>
     </inertial>
   </link>
-  <joint name="lidar_joint" type="fixed">
+  <joint name="ouster_joint" type="fixed">
     <parent link="base_link"/>
-    <child link="lidar_link"/>
-    <origin xyz="0.1 0.0 0.03" rpy="0 0 0"/>
+    <child link="ouster_link"/>
+    <origin xyz="0.0 0.0 0.30" rpy="0 0 0"/>
   </joint>
-    <gazebo reference="lidar_link">
-    <sensor name="lidar" type="gpu_lidar">
+    <gazebo reference="ouster_link">
+    <sensor name="ouster" type="gpu_lidar">
         <always_on>1</always_on>
-        <update_rate>5</update_rate>
-        <topic>scan</topic>
-        <gz_frame_id>lidar_link</gz_frame_id>
+        <update_rate>10</update_rate>
+        <topic>ouster/points</topic>
+        <gz_frame_id>ouster_link</gz_frame_id>
         <lidar>
         <scan>
             <horizontal>
-            <samples>180</samples>
+            <samples>1024</samples>
             <resolution>1</resolution>
             <min_angle>-3.14159</min_angle>
             <max_angle>3.14159</max_angle>
             </horizontal>
+            <vertical>
+            <samples>16</samples>
+            <resolution>1</resolution>
+            <min_angle>-0.261799</min_angle>
+            <max_angle>0.261799</max_angle>
+            </vertical>
         </scan>
         <range>
-            <min>0.1</min>
-            <max>10.0</max>
-            <resolution>0.01</resolution>
+            <min>0.3</min>
+            <max>20.0</max>
+            <resolution>0.02</resolution>
         </range>
         </lidar>
         <visualize>false</visualize>
     </sensor>
-    </gazebo> -->
+    </gazebo>
     <gazebo>
       <plugin

Commit message: bringup: lower ouster mount and publish debug map frame

File: src/lunabot_description/urdf/lunabot.urdf.xacro (robot description, xacro)
@@ -20,5 +20,5 @@
     <parent link="base_link"/>
     <child link="ouster_link"/>
-    <origin xyz="0.0 0.0 0.30" rpy="0 0 0"/>
+    <origin xyz="0.0 0.0 0.06" rpy="0 0 0"/>
   </joint>
     <gazebo reference="ouster_link">

Commit message: sim: raise ouster mount above front camera

File: src/lunabot_description/urdf/lunabot.urdf.xacro (robot description, xacro)
@@ -20,5 +20,5 @@
     <parent link="base_link"/>
     <child link="ouster_link"/>
-    <origin xyz="0.0 0.0 0.06" rpy="0 0 0"/>
+    <origin xyz="0.0 0.0 0.10" rpy="0 0 0"/>
   </joint>
     <gazebo reference="ouster_link">

Commit message: sim: nudge ouster mount higher for front clearance

File: src/lunabot_description/urdf/lunabot.urdf.xacro (robot description, xacro)
@@ -20,5 +20,5 @@
     <parent link="base_link"/>
     <child link="ouster_link"/>
-    <origin xyz="0.0 0.0 0.10" rpy="0 0 0"/>
+    <origin xyz="0.0 0.0 0.12" rpy="0 0 0"/>
   </joint>
     <gazebo reference="ouster_link">

Commit message: Feat/lidar nav2 costmaps (#133)
* nav2: switch costmaps to ouster point cloud

* bringup: add lidar-only nav debug mode

* nav2: drop explicit costmap geometry in debug mode

* nav2: publish full costmaps and densify lidar sim

* bringup: lower ouster mount and publish debug map frame

* sim: raise ouster mount above front camera

* sim: nudge ouster mount higher for front clearance

File: src/lunabot_description/urdf/lunabot.urdf.xacro (robot description, xacro)
@@ -20,5 +20,5 @@
     <parent link="base_link"/>
     <child link="ouster_link"/>
-    <origin xyz="0.0 0.0 0.30" rpy="0 0 0"/>
+    <origin xyz="0.0 0.0 0.12" rpy="0 0 0"/>
   </joint>
     <gazebo reference="ouster_link">
@@ -37,5 +37,5 @@
             </horizontal>
             <vertical>
-            <samples>16</samples>
+            <samples>32</samples>
             <resolution>1</resolution>
             <min_angle>-0.261799</min_angle>
@@ -44,5 +44,5 @@
         </scan>
         <range>
-            <min>0.3</min>
+            <min>0.1</min>
             <max>20.0</max>
             <resolution>0.02</resolution>

Commit message: fix: raise camera and lidar mounts for better ground separation
Camera: 0.05m → 0.30m above base_link (~0.50m above ground), pitch
reduced from 17° to 15°. Higher mount gives cleaner angular separation
between ground plane and obstacles in the depth point cloud, making the
costmap min_obstacle_height filter far more reliable.

Ouster: 0.12m → 0.35m above base_link (~0.55m above ground). Highest
point on the rover for unobstructed 360° coverage.

Made-with: Cursor

File: src/lunabot_description/urdf/lunabot.urdf.xacro (robot description, xacro)
@@ -20,5 +20,5 @@
     <parent link="base_link"/>
     <child link="ouster_link"/>
-    <origin xyz="0.0 0.0 0.12" rpy="0 0 0"/>
+    <origin xyz="0.0 0.0 0.35" rpy="0 0 0"/>
   </joint>
     <gazebo reference="ouster_link">
@@ -87,5 +87,5 @@
       <parent link="base_link" />
       <child link="camera_front_link" />
-      <origin xyz="0.12 0.0 0.05" rpy="0 0.3 0" />
+      <origin xyz="0.12 0.0 0.30" rpy="0 0.26 0" />
     </joint>
     <link name="camera_front_optical_frame" />

Commit message: fix: strip costmaps back to proven working PR #117 config
Revert to the simple ObstacleLayer + raw PointCloud2 approach that
worked reliably in PR #117. Remove the VoxelLayer, depthimage_to_
laserscan middleman, and complex multi-layer setup that produced
phantom obstacles and unusable costmaps.

- Camera back to 5cm above base_link with 0.3 rad pitch
- Both costmaps use a single ObstacleLayer fed by /camera_front/points
- max_obstacle_height 0.45m, min_obstacle_height 0.10m
- Global costmap keeps RTAB-Map static_layer for the /map grid
- Remove depthimage_to_laserscan node from navigation launch
- Revert RTAB-Map Grid/MaxGroundHeight to 0.10

File: src/lunabot_description/urdf/lunabot.urdf.xacro (robot description, xacro)
@@ -87,5 +87,5 @@
       <parent link="base_link" />
       <child link="camera_front_link" />
-      <origin xyz="0.12 0.0 0.30" rpy="0 0.26 0" />
+      <origin xyz="0.12 0.0 0.05" rpy="0 0.3 0" />
     </joint>
     <link name="camera_front_optical_frame" />

Commit message: Replace global EKF with RTAB-Map SLAM for map->odom drift correction (#226)
* Replace global EKF with RTAB-Map SLAM for map->odom correction

The dual-EKF architecture (local + global) suffered from continuous drift
because the global EKF had no persistent correction source after the
initial AprilTag seed. This made the arena appear to swim relative to
the rover during multi-waypoint traversals.

RTAB-Map SLAM now owns the map->odom transform via visual loop closure
and AprilTag landmark constraints. The local EKF continues to provide
smooth odom->base_footprint from wheel odometry + IMU. This matches
the architecture used by College of DuPage and Chicago Robotics teams.

Changes:
- rtabmap.yaml: subscribe_depth=true, publish_tf=true, no internal VO
- ekf.yaml: removed ekf_filter_node_map section entirely
- localisation.launch.py: removed global EKF node, rgbd_odometry node,
  and enable_visual_slam flag; RTAB-Map always active in normal mode;
  tag_detections remapped to /camera_front/tags for landmark support
- start_zone_localiser.py: removed all SetPose/global EKF interaction;
  transitions directly to READY once stable tag lock is acquired
- Deleted dead code: visual_odometry_gate.py, stereo_camera_info_publisher.py
- Updated tests, config, README, package.xml, setup.py

Made-with: Cursor

* fix: use RTAB-Map cloud_obstacles for costmaps instead of raw points

Raw point clouds from the depth camera include the ground plane, which
the costmap interprets as obstacles — filling the map with black cells.

Switch both global and local costmaps to subscribe to /cloud_obstacles
from RTAB-Map, which applies ground/obstacle segmentation via Grid/*
parameters (MaxGroundAngle, MaxGroundHeight, MinClusterSize, etc.).
This is the same pattern used by College of DuPage and EDT teams.

Also replace the 2D ObstacleLayer with VoxelLayer for proper 3D
height filtering of the segmented obstacle cloud.

Made-with: Cursor

* fix: increase RTAB-Map sync tolerance for Gazebo timing

RTAB-Map was failing to look up odom->base_footprint TF for every image
frame because the camera image timestamps were slightly behind the TF
buffer, especially after Gazebo sim-time jumps during startup.

Increase wait_for_transform from 0.2s to 1.0s and relax
approx_sync_max_interval from 0.02s to 0.1s.

Made-with: Cursor

* fix: use raw camera points with height-based ground filter for costmaps

RTAB-Map's /cloud_obstacles was not publishing because Gazebo sim-time
jumps kept clearing the TF buffer, preventing frame processing.

Switch to /camera_front/points directly with min_obstacle_height 0.15m
(camera is at 0.248m; ground in base_footprint frame is z≈0). This
removes the RTAB-Map dependency for costmap obstacle detection and works
independently of SLAM timing issues.

Made-with: Cursor

* fix: raise camera and lidar mounts for better ground separation

Camera: 0.05m → 0.30m above base_link (~0.50m above ground), pitch
reduced from 17° to 15°. Higher mount gives cleaner angular separation
between ground plane and obstacles in the depth point cloud, making the
costmap min_obstacle_height filter far more reliable.

Ouster: 0.12m → 0.35m above base_link (~0.55m above ground). Highest
point on the rover for unobstructed 360° coverage.

Made-with: Cursor

* fix: set Grid/Sensor to 0 (depth) to match FromDepth mode

Grid/Sensor=2 expects a 3D lidar scan topic which is not subscribed,
causing "Cannot create local map from scan: scan is empty" warnings.
Sensor=0 uses the subscribed depth image for grid generation.

* fix: replace VoxelLayer with depthimage_to_laserscan for costmaps

Raw depth point clouds into VoxelLayer caused ghost obstacles because:
- ground plane noise passed through height threshold filters
- no clearing mechanism for stale obstacles (no inf rays in PointCloud2)
- RTAB-Map cloud_obstacles accumulates permanently with no clearing

New architecture (matches COD/EDT/community best practices):
- depthimage_to_laserscan converts depth image to virtual LaserScan
- Local costmap: ObstacleLayer from /depth_scan with inf_is_valid=true
  for proper clearing of empty space
- Global costmap: StaticLayer only, fed by RTAB-Map's /map occupancy grid

* fix: correct depthimage_to_laserscan param name to output_frame

The parameter was incorrectly named output_frame_id (doesn't exist),
causing the scan to publish in the default camera_depth_frame which
has no TF entry. The correct parameter name is output_frame.

* fix: remap RTAB-Map /map output to avoid overriding map_server

RTAB-Map was publishing its small explored map on /map, overriding
the map_server's arena-sized blank map. The global costmap's static
layer received the tiny RTAB-Map map (~1.5m) instead of the 14x14m
blank arena map, making path planning impossible.

* fix: overhaul costmap architecture based on COD reference

- Let RTAB-Map publish /map directly (remove blank map_server)
- Add obstacle_layer + voxel_layer to BOTH global and local costmaps
- Global costmap: static_layer (RTAB-Map) + obstacle + voxel + inflation
- Local costmap: obstacle + voxel + inflation
- Fix inf_is_valid to false (was erasing obstacles with inf rays)
- Increase inflation radius from 0.30m to 0.55m
- Increase scan_height from 60 to 200 rows (catch low obstacles)
- Reduce range_max from 4.0 to 3.0m (less noise at long range)
- Add behavior_server, velocity_smoother, waypoint_follower configs
- Add RTAB-Map: LinearUpdate, AngularUpdate, StartAtOrigin, GridGlobal

Architecture modeled after College of DuPage Lunabotics team (Nav2 +
RTAB-Map + depth cameras). Their repo: research/lunabot_ros

* fix: obstacle_layer clears only, voxel_layer marks with height filter

The downward-pitched camera produces LaserScan rays that hit the
ground at 0.3-0.5m, flooding the costmap with false obstacles.

- obstacle_layer: marking=false, clearing=true (raytrace clear only)
- voxel_layer: marking=true, clearing=true, min_obstacle_height=0.10
  (filters ground returns, only marks objects >10cm above ground)

* fix: raise ground filter to 0.15m, disable start-zone spin

- Bump min_obstacle_height from 0.10 to 0.15 on both global and local
  voxel_layer to stop Gazebo ground mesh being marked as obstacles
- Raise RTAB-Map Grid/MaxGroundHeight from 0.10 to 0.15 to match
- Set start_zone_localiser angular speeds to 0.0 so it no longer
  rotates the rover while searching for the AprilTag

* fix: update preflight config for current architecture

Remove ekf_filter_node_map and map_server from required nodes (both
removed from the stack). Mark /map, /ouster/points and map->odom TF
as non-critical since RTAB-Map takes time to produce the first map.

* fix: strip costmaps back to proven working PR #117 config

Revert to the simple ObstacleLayer + raw PointCloud2 approach that
worked reliably in PR #117. Remove the VoxelLayer, depthimage_to_
laserscan middleman, and complex multi-layer setup that produced
phantom obstacles and unusable costmaps.

- Camera back to 5cm above base_link with 0.3 rad pitch
- Both costmaps use a single ObstacleLayer fed by /camera_front/points
- max_obstacle_height 0.45m, min_obstacle_height 0.10m
- Global costmap keeps RTAB-Map static_layer for the /map grid
- Remove depthimage_to_laserscan node from navigation launch
- Revert RTAB-Map Grid/MaxGroundHeight to 0.10

* fix: use absolute path for Nav2 BT XML

The short filename does not resolve; provide the full installed path.

* fix: restore gz_frame_id to camera_front_link

The optical frame has REP-103 rotations that flip the point cloud
90 degrees sideways. PR #117 used camera_front_link and worked.

* chore: clean up stale references to removed nodes

- Remove ekf_filter_node_map TF contract (RTAB-Map owns map->odom now)
- Replace map_server with rtabmap in lidar-debug and dry-run preflight
- Remove depthimage_to_laserscan exec_depend from bringup package.xml
- Fix README indentation flagged by CodeRabbit

File: src/lunabot_description/urdf/lunabot.urdf.xacro (robot description, xacro)
@@ -20,5 +20,5 @@
     <parent link="base_link"/>
     <child link="ouster_link"/>
-    <origin xyz="0.0 0.0 0.12" rpy="0 0 0"/>
+    <origin xyz="0.0 0.0 0.35" rpy="0 0 0"/>
   </joint>
     <gazebo reference="ouster_link">
@@ -112,5 +112,5 @@
       <update_rate>15</update_rate>
       <topic>camera_front</topic>
-      <gz_frame_id>camera_front_optical_frame</gz_frame_id>
+      <gz_frame_id>camera_front_link</gz_frame_id>
       </sensor>
     </gazebo>

Commit message: feat: add rear depth camera to URDF and simulation bridge
Mirrors the front OAK-D camera at the back of the rover for the shuttle
drive strategy.  The rear camera provides obstacle detection when
reversing, eliminating the need for 180-degree turns.

Closes #238

File: src/lunabot_description/urdf/lunabot.urdf.xacro (robot description, xacro)
@@ -115,3 +115,54 @@
       </sensor>
     </gazebo>
+    <!-- Rear depth camera — mirrors the front camera for reverse-drive obstacle
+         detection in the shuttle drive strategy. -->
+    <link name="camera_rear_link">
+    <visual>
+      <geometry>
+        <cylinder length="0.05" radius="0.03" />
+      </geometry>
+      <material name="dark_grey">
+        <color rgba="0.2 0.2 0.2 1.0" />
+      </material>
+    </visual>
+    <collision>
+      <geometry>
+        <cylinder length="0.05" radius="0.03" />
+      </geometry>
+    </collision>
+    <inertial>
+      <mass value="0.1" />
+      <inertia ixx="0.0001" ixy="0" ixz="0" iyy="0.0001" iyz="0" izz="0.0001" />
+    </inertial>
+  </link>
+    <joint name="camera_rear_joint" type="fixed">
+      <parent link="base_link" />
+      <child link="camera_rear_link" />
+      <origin xyz="-0.12 0.0 0.05" rpy="0 0.3 ${pi}" />
+    </joint>
+    <link name="camera_rear_optical_frame" />
+    <joint name="camera_rear_optical_joint" type="fixed">
+      <parent link="camera_rear_link" />
+      <child link="camera_rear_optical_frame" />
+      <origin xyz="0 0 0" rpy="-${pi/2} 0.0 -${pi/2}" />
+    </joint>
+    <gazebo reference="camera_rear_link">
+      <sensor name="camera_rear" type="rgbd_camera">
+      <camera>
+        <horizontal_fov>1.57</horizontal_fov>
+        <image>
+          <width>640</width>
+          <height>480</height>
+        </image>
+        <clip>
+          <near>0.1</near>
+          <far>10</far>
+        </clip>
+      </camera>
+      <always_on>1</always_on>
+      <update_rate>15</update_rate>
+      <topic>camera_rear</topic>
+      <gz_frame_id>camera_rear_link</gz_frame_id>
+      </sensor>
+    </gazebo>
 </robot>
